File: osnova8 project/Schematics/KiCad/Osnova8/Osnova8.kicad_sch (KiCad schematic)
At the start: 0 parts

Commit message: updated schematics
Other:
- sheet COMLOG renamed CMBL
- sheet SCTPS renamed SFPS
Changed lines of the file:
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@@
 			(color 0 0 0 0.0000)
 		)
-		(property "Sheetname" "COMLOG"
+		(property "Sheetname" "CMBL"
 			(at 30.48 99.6184 0)
 			(effects
@@
 			(color 0 0 0 0.0000)
 		)
-		(property "Sheetname" "SCTPS"
+		(property "Sheetname" "SFPS"
 			(at 30.48 46.2784 0)
 			(effects
