File: osnova8 project/Schematics/KiCad/Osnova8/Osnova8_IEU.kicad_sch (KiCad schematic)
At the start: 16 parts, among them U10 74LS138, U11 74LS138, U12 74LS138, U13 74LS161, U14 74LS161, U15 74LS541, U8 74LS374, U9 74LS138

Commit message: updated schematics
Parts:
- removed C15: C, symbol Device:C
- removed U12: 74LS138, symbol 74xx:74LS138
Connections:
- net ARG_DVR: now also U15.1 (G1)
- net GNDREF: now also U11.6 (E3), U15.19 (G2); no longer U10.5 (E2), U11.4 (E1), U11.5 (E2), U9.5 (E2)
- net OPC0: now reaches U10.1 (A0), U11.1 (A0), U8.12 (O4)
- net OPC1: now reaches U10.2 (A1), U11.2 (A1), U8.15 (O5)
- net OPC2: now reaches U10.3 (A2), U11.3 (A2), U8.16 (O6)
- net OPC3: now reaches U10.4 (E1), U8.19 (O7)
- net OPC3: now also U11.5 (E2); no longer U11.6 (E3)
- net DIR7: now reaches U13.11 (Q3), U15.9 (A7)
- net DIR6: now reaches U13.12 (Q2), U15.8 (A6)
- net ARG_SCTSPS renamed ARG_SFPS
- net OPC_INTSO renamed OPC_INTSX
- net OPC_SCT renamed OPC_SF
- new net ACT_INST: U9.5 (E2)
- new net ACT_OPC: U10.5 (E2), U11.4 (E1)
