File: osnova8 project/Schematics/KiCad/Osnova8/Osnovca_ALU.kicad_sch (KiCad schematic)
At the start: 14 parts, among them U1 74LS181, U2 74LS181, U3 74LS374, U4 74LS374, U5 74LS541, U6 74LS374, U7 74LS374

Commit message: updated schematics
Connections:
- net ARG_RES renamed ARG_RESR
- net DIR0 renamed DVR0
- net DIR1 renamed DVR1
- net DIR2 renamed DVR2
- net DIR3 renamed DVR3
- net DIR4 renamed DVR4
- net DIR5 renamed DVR5
- net OPC_RES renamed OPC_RESR
Changed lines of the file:
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@@
 	(title_block
 		(title "Osnova8 CPU")
-		(date "2025-12-03")
+		(date "2026-01-13")
+		(rev "2")
 	)
 	(junction
@@
 	(wire
 		(pts
-			(xy 96.52 172.72) (xy 99.06 172.72)
-		)
-		(stroke
-			(width 0)
-			(type default)
-		)
-	)
-	(wire
-		(pts
 			(xy 168.91 107.95) (xy 125.73 107.95)
 		)
@@
 	(wire
 		(pts
-			(xy 96.52 170.18) (xy 99.06 170.18)
-		)
-		(stroke
-			(width 0)
-			(type default)
-		)
-	)
-	(wire
-		(pts
 			(xy 115.57 105.41) (xy 99.06 105.41)
 		)
@@
 	(wire
 		(pts
+			(xy 96.52 172.72) (xy 99.06 172.72)
+		)
+		(stroke
+			(width 0)
+			(type default)
+		)
+	)
+	(wire
+		(pts
 			(xy 135.89 39.37) (xy 168.91 39.37)
 		)
@@
 	(wire
 		(pts
+			(xy 96.52 170.18) (xy 99.06 170.18)
+		)
+		(stroke
+			(width 0)
+			(type default)
+		)
+	)
+	(wire
+		(pts
 			(xy 133.35 39.37) (xy 133.35 100.33)
 		)
@@
 		)
 	)
-	(global_label "DIR1"
+	(global_label "DVR1"
 		(shape bidirectional)
 		(at 146.05 123.19 180)
@@
 		)
 		(property "Intersheetrefs" "${INTERSHEET_REFS}"
-			(at 139.2897 123.19 0)
+			(at 137.1154 123.19 0)
 			(effects
 				(font
@@
 		)
 	)
-	(global_label "DIR4"
+	(global_label "DVR4"
 		(shape bidirectional)
 		(at 166.37 64.77 180)
@@
 		)
 		(property "Intersheetrefs" "${INTERSHEET_REFS}"
-			(at 159.6097 64.77 0)
+			(at 157.4354 64.77 0)
 			(effects
 				(font
@@
 		)
 	)
-	(global_label "ARG_RES"
+	(global_label "ARG_RESR"
 		(shape bidirectional)
-		(at 96.8386 172.72 180)
+		(at 96.52 172.72 180)
 		(fields_autoplaced yes)
 		(effects
@@
 		)
 		(property "Intersheetrefs" "${INTERSHEET_REFS}"
-			(at 86.9819 172.72 0)
+			(at 82.9288 172.72 0)
 			(effects
 				(font
@@
 		)
 	)
-	(global_label "DIR0"
+	(global_label "DVR0"
 		(shape bidirectional)
 		(at 146.05 120.65 180)
@@
 		)
 		(property "Intersheetrefs" "${INTERSHEET_REFS}"
-			(at 139.2897 120.65 0)
+			(at 137.1154 120.65 0)
 			(effects
 				(font
@@
 		)
 	)
-	(global_label "OPC_RES"
+	(global_label "OPC_RESR"
 		(shape bidirectional)
-		(at 96.8386 170.18 180)
+		(at 96.52 170.18 180)
 		(fields_autoplaced yes)
 		(effects
@@
 		)
 		(property "Intersheetrefs" "${INTERSHEET_REFS}"
-			(at 86.7884 170.18 0)
+			(at 82.6869 170.18 0)
 			(effects
 				(font
@@
 		)
 	)
-	(global_label "DIR2"
+	(global_label "DVR2"
 		(shape bidirectional)
 		(at 146.05 125.73 180)
@@
 		)
 		(property "Intersheetrefs" "${INTERSHEET_REFS}"
-			(at 139.2897 125.73 0)
+			(at 137.1154 125.73 0)
 			(effects
 				(font
@@
 		)
 	)
-	(global_label "DIR3"
+	(global_label "DVR3"
 		(shape bidirectional)
 		(at 146.05 128.27 180)
@@
 		)
 		(property "Intersheetrefs" "${INTERSHEET_REFS}"
-			(at 139.2897 128.27 0)
+			(at 137.1154 128.27 0)
 			(effects
 				(font
@@
 		)
 	)
-	(global_label "DIR5"
+	(global_label "DVR5"
 		(shape bidirectional)
 		(at 146.05 133.35 180)
@@
 		)
 		(property "Intersheetrefs" "${INTERSHEET_REFS}"
-			(at 139.2897 133.35 0)
+			(at 137.1154 133.35 0)
 			(effects
 				(font
